Commit message: Remaping topic

File: src/my_r2d2/urdf/r2d2.urdf (robot description, URDF)
Before this commit: robot R2D2, 7 links, 6 joints
Links:
- added link box, mass 1; collision box size=.08 .08 .08; visual box size=.08 .08 .08
- added link left_back_wheel, mass 1; collision cylinder length=0.1 radius=0.035; visual cylinder length=0.1 radius=0.035
- added link left_base, mass 10; collision box size=0.4 .1 .1; visual box size=0.4 .1 .1
- added link left_front_wheel, mass 1; collision cylinder length=0.1 radius=0.035; visual cylinder length=0.1 radius=0.035
- added link left_tip, mass 0.05; collision mesh filename=package://pr2_description/meshes/gripper_v0/l_finger_tip.dae; visual mesh filename=package://pr2_description/meshes/gripper_v0/l_finger_tip.dae
- added link right_back_wheel, mass 1; collision cylinder length=0.1 radius=0.035; visual cylinder length=0.1 radius=0.035
- added link right_base, mass 10; collision box size=0.4 .1 .1; visual box size=0.4 .1 .1
- added link right_front_wheel, mass 1; collision cylinder length=0.1 radius=0.035; visual cylinder length=0.1 radius=0.035
- added link right_tip, mass 0.05; collision mesh filename=package://pr2_description/meshes/gripper_v0/l_finger_tip.dae; visual mesh filename=package://pr2_description/meshes/gripper_v0/l_finger_tip.dae
- link gripper_pole: mass None -> 0.05; geometry collision cylinder length=0.2 radius=.01; visual cylinder length=0.2 radius=.01
- link head: mass None -> 2; geometry collision sphere radius=0.2; visual sphere radius=0.2
- link left_gripper: mass None -> 0.05; geometry collision mesh filename=package://pr2_description/meshes/gripper_v0/l_finger.dae; visual mesh filename=package://pr2_description/meshes/gripper_v0/l_finger.dae
- link left_leg: mass None -> 10; geometry collision box size=0.6 .1 .2; visual box size=0.6 .1 .2
- link right_gripper: mass None -> 0.05; geometry collision mesh filename=package://pr2_description/meshes/gripper_v0/l_finger.dae; visual mesh filename=package://pr2_description/meshes/gripper_v0/l_finger.dae
- link right_leg: mass None -> 10; geometry collision box size=0.6 .1 .2; visual box size=0.6 .1 .2
Joints:
- added joint left_back_wheel_joint: type continuous, parent left_base, child left_back_wheel, origin xyz=-0.133333333333 0 -0.085 rpy=0 0 0, axis 0 1 0
- added joint left_base_joint: type fixed, parent left_leg, child left_base, origin xyz=0 0 -0.6
- added joint left_front_wheel_joint: type continuous, parent left_base, child left_front_wheel, origin xyz=0.133333333333 0 -0.085 rpy=0 0 0, axis 0 1 0
- added joint left_tip_joint: type fixed, parent left_gripper, child left_tip
- added joint right_back_wheel_joint: type continuous, parent right_base, child right_back_wheel, origin xyz=-0.133333333333 0 -0.085 rpy=0 0 0, axis 0 1 0
- added joint right_base_joint: type fixed, parent right_leg, child right_base, origin xyz=0 0 -0.6
- added joint right_front_wheel_joint: type continuous, parent right_base, child right_front_wheel, origin xyz=0.133333333333 0 -0.085 rpy=0 0 0, axis 0 1 0
- added joint right_tip_joint: type fixed, parent right_gripper, child right_tip
- added joint tobox: type fixed, parent head, child box, origin xyz=0.1814 0 0.1414
- joint base_to_left_leg: origin xyz=-0.22 0 .25 -> xyz=0 0.22 .25
- joint base_to_right_leg: origin xyz=0.22 0 .25 -> xyz=0 -0.22 .25
- joint gripper_extension: origin xyz=0 0.19 .2 rpy=0 0 1.57075 -> xyz=0.19 0 .2 rpy=0 0 0
- joint right_gripper_joint: axis 0 0 1 -> 0 0 -1; limit lower=0.0 upper=-0.548 effort=1000.0 velocity=0.5 -> lower=0.0 upper=0.548 effort=1000.0 velocity=0.5; origin xyz=0.2 0.01 0 rpy=0 0 0 -> xyz=0.2 -0.01 0 rpy=0 0 0
