Commit message: Markers and camera

File: src/my_r2d2/urdf/r2d2.urdf.xacro (robot description, xacro)
@@ -220,3 +220,10 @@
     <origin xyz="0 0 ${wheeldiam + bodylen/2 + .1}"/>
   </joint>
+  <link name="eye">
+  </link>
+  <joint name="box_eye_link" type="fixed">
+    <parent link="box"/>
+    <child link="eye"/>
+    <origin rpy="${pi/2} ${pi} ${pi/2}"/>
+  </joint>
 </robot>
